File: hardware/drone_esc/schematics/mcu_2.kicad_sch (KiCad schematic)
At the start: 0 parts

Commit message: finished 4 esc schematics need further refinment of the sheets
Parts:
- added C18: 4.7uF 10V X7R MLCC, Capacitor_SMD:C_0603_1608Metric, symbol Device:C
- added C19: 100nF 16V X7R MLCC, Capacitor_SMD:C_01005_0402Metric, symbol Device:C
- added C20: 100nF 10V X7R MLCC, Capacitor_SMD:C_0402_1005Metric, symbol Device:C
- added TP5: DShot, Drone_components:Rectangle test point, symbol Drone_components:Rectangle_test_point
- added TP6: ~, Drone_components:1.27 test pad, symbol Drone_components:1.27_test_pad
- added U5: STM32G071GBU6, Package_DFN_QFN:QFN-28_4x4mm_P0.5mm, symbol MCU_ST_STM32G0:STM32G071GBUxN
Connections:
- new net: TP5.1, U5.28 (PB8)
- new net: C19.2, U5.5 (PF2)
- new net +3.3V: C18.1, C20.1, TP6.1 (V), U5.3 (VDD)
- new net GND: C18.2, C19.1, C20.2, TP6.4 (GND), U5.4 (VSS)
- new net HIN2A: U5.19 (PA10/PA12)
- new net HIN2B: U5.18 (PA9/PA11)
- new net HIN2C: U5.16 (PA8)
- new net LIN2A: U5.15 (PB15)
- new net LIN2B: U5.14 (PB0)
- new net LIN2C: U5.13 (PA7)
- new net SWCLK: TP6.3 (SWCLK), U5.21 (PA14)
- new net SWDIO: TP6.2 (SWDIO), U5.20 (PA13)
- new net VSense2A: U5.6 (PA0)
- new net VSense2B: U5.7 (PA1)
- new net VSense2C: U5.8 (PA2)
- no-connect marks 0 -> 13
Other:
- note added: "STM32G071GBU6"
- note added: "SWD Debugging"

Commit message: finnished component placement
Parts:
- C18: value 4.7uF 10V X7R MLCC -> 4.7uF 10V X5R MLCC; footprint Capacitor_SMD:C_0603_1608Metric -> Capacitor_SMD:C_0402_1005Metric; JLCPCB part C108342 -> C23733
- C19: footprint Capacitor_SMD:C_01005_0402Metric -> Capacitor_SMD:C_0402_1005Metric
Changed lines of the file:
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@@
 			)
 		)
-		(property "Footprint" "Capacitor_SMD:C_01005_0402Metric"
+		(property "Footprint" "Capacitor_SMD:C_0402_1005Metric"
 			(at 87.63 129.8448 0)
 			(effects
@@
 			)
 		)
-		(property "Value" "4.7uF 10V X7R MLCC"
+		(property "Value" "4.7uF 10V X5R MLCC"
 			(at 64.77 115.5699 0)
 			(effects
@@
 			)
 		)
-		(property "Footprint" "Capacitor_SMD:C_0603_1608Metric"
+		(property "Footprint" "Capacitor_SMD:C_0402_1005Metric"
 			(at 61.9252 118.11 0)
 			(effects
@@
 			)
 		)
-		(property "JLCPCB part" "C108342"
+		(property "JLCPCB part" "C23733"
 			(at 60.96 114.3 0)
 			(effects
