File: hardware/drone_esc/schematics/mcu_3.kicad_sch (KiCad schematic)
At the start: 0 parts

Commit message: finished 4 esc schematics need further refinment of the sheets
Parts:
- added C41: 4.7uF 10V X7R MLCC, Capacitor_SMD:C_0603_1608Metric, symbol Device:C
- added C42: 100nF 16V X7R MLCC, Capacitor_SMD:C_01005_0402Metric, symbol Device:C
- added C43: 100nF 10V X7R MLCC, Capacitor_SMD:C_0402_1005Metric, symbol Device:C
- added TP7: DShot, Drone_components:Rectangle test point, symbol Drone_components:Rectangle_test_point
- added TP8: ~, Drone_components:1.27 test pad, symbol Drone_components:1.27_test_pad
- added U8: STM32G071GBU6, Package_DFN_QFN:QFN-28_4x4mm_P0.5mm, symbol MCU_ST_STM32G0:STM32G071GBUxN
Connections:
- new net: TP7.1, U8.28 (PB8)
- new net: C42.2, U8.5 (PF2)
- new net +3.3V: C41.1, C43.1, TP8.1 (V), U8.3 (VDD)
- new net GND: C41.2, C42.1, C43.2, TP8.4 (GND), U8.4 (VSS)
- new net HIN3A: U8.19 (PA10/PA12)
- new net HIN3B: U8.18 (PA9/PA11)
- new net HIN3C: U8.16 (PA8)
- new net LIN3A: U8.15 (PB15)
- new net LIN3B: U8.14 (PB0)
- new net LIN3C: U8.13 (PA7)
- new net SWCLK: TP8.3 (SWCLK), U8.21 (PA14)
- new net SWDIO: TP8.2 (SWDIO), U8.20 (PA13)
- new net VSense3A: U8.6 (PA0)
- new net VSense3B: U8.7 (PA1)
- new net VSense3C: U8.8 (PA2)
- no-connect marks 0 -> 13
Other:
- note added: "STM32G071GBU6"
- note added: "SWD Debugging"

Commit message: finnished component placement
Parts:
- C41: value 4.7uF 10V X7R MLCC -> 4.7uF 10V X5R MLCC; footprint Capacitor_SMD:C_0603_1608Metric -> Capacitor_SMD:C_0402_1005Metric; JLCPCB part C108342 -> C23733
- C42: footprint Capacitor_SMD:C_01005_0402Metric -> Capacitor_SMD:C_0402_1005Metric
Changed lines of the file:
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@@
+	)
+	(symbol
+		(lib_id "power:GND")
+		(at 60.96 120.65 0)
+		(unit 1)
+		(exclude_from_sim no)
+		(in_bom yes)
+		(on_board yes)
+		(dnp no)
+		(fields_autoplaced yes)
+		(property "Reference" "#PWR054"
+			(at 60.96 127 0)
+			(effects
+				(font
+					(size 1.27 1.27)
+				)
+				(hide yes)
+			)
+		)
+		(property "Value" "GND"
+			(at 60.96 125.73 0)
+			(effects
+				(font
+					(size 1.27 1.27)
+				)
+			)
+		)
+		(property "Footprint" ""
+			(at 60.96 120.65 0)
+			(effects
+				(font
+					(size 1.27 1.27)
+				)
+				(hide yes)
+			)
+		)
+		(property "Datasheet" ""
+			(at 60.96 120.65 0)
+			(effects
+				(font
+					(size 1.27 1.27)
+				)
+				(hide yes)
+			)
+		)
+		(property "Description" "Power symbol creates a global label with name \"GND\" , ground"
+			(at 60.96 120.65 0)
+			(effects
+				(font
+					(size 1.27 1.27)
+				)
+				(hide yes)
+			)
+		)
+		(pin "1"
+		)
+		(instances
+			(project "drone_esc"
+				(path "/b5a13fd4-6868-4fff-a56c-eae40f1d53c7/189a97be-36f6-4952-93ff-62f3a17cbe5b"
+					(reference "#PWR054")
+					(unit 1)
+				)
+			)
+		)
 	)
 	(symbol
@@
 			)
 		)
-		(property "Value" "4.7uF 10V X7R MLCC"
+		(property "Value" "4.7uF 10V X5R MLCC"
 			(at 64.77 115.5699 0)
 			(effects
@@
 			)
 		)
-		(property "Footprint" "Capacitor_SMD:C_0603_1608Metric"
+		(property "Footprint" "Capacitor_SMD:C_0402_1005Metric"
 			(at 61.9252 118.11 0)
 			(effects
@@
 			)
 		)
-		(property "JLCPCB part" "C108342"
+		(property "JLCPCB part" "C23733"
 			(at 60.96 114.3 0)
 			(effects
@@
 				(path "/b5a13fd4-6868-4fff-a56c-eae40f1d53c7/189a97be-36f6-4952-93ff-62f3a17cbe5b"
 					(reference "C41")
-					(unit 1)
-				)
-			)
-		)
-	)
-	(symbol
-		(lib_id "power:GND")
-		(at 60.96 120.65 0)
-		(unit 1)
-		(exclude_from_sim no)
-		(in_bom yes)
-		(on_board yes)
-		(dnp no)
-		(fields_autoplaced yes)
-		(property "Reference" "#PWR054"
-			(at 60.96 127 0)
-			(effects
-				(font
-					(size 1.27 1.27)
-				)
-				(hide yes)
-			)
-		)
-		(property "Value" "GND"
-			(at 60.96 125.73 0)
-			(effects
-				(font
-					(size 1.27 1.27)
-				)
-			)
-		)
-		(property "Footprint" ""
-			(at 60.96 120.65 0)
-			(effects
-				(font
-					(size 1.27 1.27)
-				)
-				(hide yes)
-			)
-		)
-		(property "Datasheet" ""
-			(at 60.96 120.65 0)
-			(effects
-				(font
-					(size 1.27 1.27)
-				)
-				(hide yes)
-			)
-		)
-		(property "Description" "Power symbol creates a global label with name \"GND\" , ground"
-			(at 60.96 120.65 0)
-			(effects
-				(font
-					(size 1.27 1.27)
-				)
-				(hide yes)
-			)
-		)
-		(pin "1"
-		)
-		(instances
-			(project "drone_esc"
-				(path "/b5a13fd4-6868-4fff-a56c-eae40f1d53c7/189a97be-36f6-4952-93ff-62f3a17cbe5b"
-					(reference "#PWR054")
 					(unit 1)
 				)
@@
 			)
 		)
-		(property "Footprint" "Capacitor_SMD:C_01005_0402Metric"
+		(property "Footprint" "Capacitor_SMD:C_0402_1005Metric"
 			(at 87.63 129.8448 0)
 			(effects
