File: hardware/drone_esc/schematics/mcu_4.kicad_sch (KiCad schematic)
At the start: 0 parts

Commit message: finished 4 esc schematics need further refinment of the sheets
Parts:
- added C44: 4.7uF 10V X7R MLCC, Capacitor_SMD:C_0603_1608Metric, symbol Device:C
- added C45: 100nF 16V X7R MLCC, Capacitor_SMD:C_01005_0402Metric, symbol Device:C
- added C46: 100nF 10V X7R MLCC, Capacitor_SMD:C_0402_1005Metric, symbol Device:C
- added TP10: ~, Drone_components:1.27 test pad, symbol Drone_components:1.27_test_pad
- added TP9: DShot, Drone_components:Rectangle test point, symbol Drone_components:Rectangle_test_point
- added U9: STM32G071GBU6, Package_DFN_QFN:QFN-28_4x4mm_P0.5mm, symbol MCU_ST_STM32G0:STM32G071GBUxN
Connections:
- new net: C45.2, U9.5 (PF2)
- new net: TP9.1, U9.28 (PB8)
- new net +3.3V: C44.1, C46.1, TP10.1 (V), U9.3 (VDD)
- new net GND: C44.2, C45.1, C46.2, TP10.4 (GND), U9.4 (VSS)
- new net HIN4A: U9.19 (PA10/PA12)
- new net HIN4B: U9.18 (PA9/PA11)
- new net HIN4C: U9.16 (PA8)
- new net LIN4A: U9.15 (PB15)
- new net LIN4B: U9.14 (PB0)
- new net LIN4C: U9.13 (PA7)
- new net SWCLK: TP10.3 (SWCLK), U9.21 (PA14)
- new net SWDIO: TP10.2 (SWDIO), U9.20 (PA13)
- new net VSense4A: U9.6 (PA0)
- new net VSense4B: U9.7 (PA1)
- new net VSense4C: U9.8 (PA2)
- no-connect marks 0 -> 13
Other:
- note added: "STM32G071GBU6"
- note added: "SWD Debugging"

Commit message: finnished component placement
Parts:
- C44: value 4.7uF 10V X7R MLCC -> 4.7uF 10V X5R MLCC; footprint Capacitor_SMD:C_0603_1608Metric -> Capacitor_SMD:C_0402_1005Metric; JLCPCB part C108342 -> C23733
- C45: footprint Capacitor_SMD:C_01005_0402Metric -> Capacitor_SMD:C_0402_1005Metric
Changed lines of the file:
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@@
+	)
+	(symbol
+		(lib_id "Device:C")
+		(at 60.96 114.3 0)
+		(unit 1)
+		(exclude_from_sim no)
+		(in_bom yes)
+		(on_board yes)
+		(dnp no)
+		(fields_autoplaced yes)
+		(property "Reference" "C44"
+			(at 64.77 113.0299 0)
+			(effects
+				(font
+					(size 1.27 1.27)
+				)
+				(justify left)
+			)
+		)
+		(property "Value" "4.7uF 10V X5R MLCC"
+			(at 64.77 115.5699 0)
+			(effects
+				(font
+					(size 1.27 1.27)
+				)
+				(justify left)
+			)
+		)
+		(property "Footprint" "Capacitor_SMD:C_0402_1005Metric"
+			(at 61.9252 118.11 0)
+			(effects
+				(font
+					(size 1.27 1.27)
+				)
+				(hide yes)
+			)
+		)
+		(property "Datasheet" "~"
+			(at 60.96 114.3 0)
+			(effects
+				(font
+					(size 1.27 1.27)
+				)
+				(hide yes)
+			)
+		)
+		(property "Description" "Unpolarized capacitor"
+			(at 60.96 114.3 0)
+			(effects
+				(font
+					(size 1.27 1.27)
+				)
+				(hide yes)
+			)
+		)
+		(property "JLCPCB part" "C23733"
+			(at 60.96 114.3 0)
+			(effects
+				(font
+					(size 1.27 1.27)
+				)
+				(hide yes)
+			)
+		)
+		(pin "2"
+		)
+		(pin "1"
+		)
+		(instances
+			(project "drone_esc"
+				(path "/b5a13fd4-6868-4fff-a56c-eae40f1d53c7/15e37512-5316-4c1c-aba7-1d8e1d7663c0"
+					(reference "C44")
+					(unit 1)
+				)
+			)
+		)
 	)
 	(symbol
@@
 	)
 	(symbol
-		(lib_id "Device:C")
-		(at 60.96 114.3 0)
-		(unit 1)
-		(exclude_from_sim no)
-		(in_bom yes)
-		(on_board yes)
-		(dnp no)
-		(fields_autoplaced yes)
-		(property "Reference" "C44"
-			(at 64.77 113.0299 0)
-			(effects
-				(font
-					(size 1.27 1.27)
-				)
-				(justify left)
-			)
-		)
-		(property "Value" "4.7uF 10V X7R MLCC"
-			(at 64.77 115.5699 0)
-			(effects
-				(font
-					(size 1.27 1.27)
-				)
-				(justify left)
-			)
-		)
-		(property "Footprint" "Capacitor_SMD:C_0603_1608Metric"
-			(at 61.9252 118.11 0)
-			(effects
-				(font
-					(size 1.27 1.27)
-				)
-				(hide yes)
-			)
-		)
-		(property "Datasheet" "~"
-			(at 60.96 114.3 0)
-			(effects
-				(font
-					(size 1.27 1.27)
-				)
-				(hide yes)
-			)
-		)
-		(property "Description" "Unpolarized capacitor"
-			(at 60.96 114.3 0)
-			(effects
-				(font
-					(size 1.27 1.27)
-				)
-				(hide yes)
-			)
-		)
-		(property "JLCPCB part" "C108342"
-			(at 60.96 114.3 0)
-			(effects
-				(font
-					(size 1.27 1.27)
-				)
-				(hide yes)
-			)
-		)
-		(pin "2"
-		)
-		(pin "1"
-		)
-		(instances
-			(project "drone_esc"
-				(path "/b5a13fd4-6868-4fff-a56c-eae40f1d53c7/15e37512-5316-4c1c-aba7-1d8e1d7663c0"
-					(reference "C44")
-					(unit 1)
-				)
-			)
-		)
-	)
-	(symbol
 		(lib_id "power:GND")
 		(at 218.44 142.24 0)
@@
 			)
 		)
-		(property "Footprint" "Capacitor_SMD:C_01005_0402Metric"
+		(property "Footprint" "Capacitor_SMD:C_0402_1005Metric"
 			(at 87.63 129.8448 0)
 			(effects
