File: hardware/drone_esc/schematics/esc_2.kicad_sch (KiCad schematic)
At the start: 0 parts

Commit message: finished 4 esc schematics need further refinment of the sheets
Parts:
- added C21, C22, C23: 47uF 35V X7R MLCC, Capacitor_SMD:C_2220_5750Metric, symbol Device:C
- added C24, C25, C26: 10nF 10V X7R MLCC, Capacitor_SMD:C_0402_1005Metric, symbol Device:C
- added C27, C29, C30: 0.47uF 25V X7R MLCC, Capacitor_SMD:C_0603_1608Metric, symbol Device:C
- added C28: 4.7uF 25V X7R MLCC, Capacitor_SMD:C_1206_3216Metric, symbol Device:C
- added D4, D5, D6: BAT165, Drone_components:BAT165, symbol Drone_components:BAT165
- added Q10, Q11, Q12, Q7, Q8, Q9: BSC016N04LS, Drone_components:BSC016N04LS, symbol Drone_components:BSC016N04LS
- added R14, R16, R17, R18, R19, R20: 33, Resistor_SMD:R_0402_1005Metric, symbol Device:R
- added R21, R23, R25: 4.7k, Resistor_SMD:R_0402_1005Metric, symbol Device:R
- added R22, R24, R26: 1k, Resistor_SMD:R_0402_1005Metric, symbol Device:R
- added U6: FD6288Q, Drone_components:FD6288Q, symbol Drone_components:FD6288Q
Connections:
- new net: C27.1, D4.1, U6.20 (VB1)
- new net: Q11.4, R19.2
- new net: C30.1, D6.1, U6.14 (VB3)
- new net: Q9.4, R17.2
- new net: C29.1, D5.1, U6.17 (VB2)
- new net: Q10.4, R18.2
- new net: Q7.4, R14.2
- new net: Q8.4, R16.2
- new net: Q12.4, R20.2
- new net GND: C21.2, C22.2, C23.2, C24.2, C25.2, C26.2, C28.1, Q10.1-3, Q12.1-3, Q8.1-3, R22.1, R24.1, R26.1, U6.25 (EXP), U6.6 (COM)
- new net HIN2A: U6.22 (HIN1)
- new net HIN2B: U6.23 (HIN2)
- new net HIN2C: U6.24 (HIN3)
- new net HO1: R14.1, U6.19 (HO1)
- new net HO2: R17.1, U6.16 (HO2)
- new net HO3: R19.1, U6.13 (HO3)
- new net LIN2A: U6.1 (LIN1)
- new net LIN2B: U6.2 (LIN2)
- new net LIN2C: U6.3 (LIN3)
- new net LO1: R16.1, U6.11 (LO1)
- new net LO2: R18.1, U6.10 (LO2)
- new net LO3: R20.1, U6.9 (LO3)
- new net VCC: C21.1, C22.1, C23.1, C28.2, D4.2, D5.2, D6.2, Q11.5-8, Q7.5-8, Q9.5-8, U6.4 (VCC)
- new net VS1: C27.2, Q7.1-3, Q8.5-8, R21.2, U6.18 (VS1)
- new net VS2: C29.2, Q10.5-8, Q9.1-3, R23.2, U6.15 (VS2)
- new net VS3: C30.2, Q11.1-3, Q12.5-8, R25.2, U6.12 (VS3)
- new net VSense2A: C24.1, R21.1, R22.2
- new net VSense2B: C25.1, R23.1, R24.2
- new net VSense2C: C26.1, R25.1, R26.2

Commit message: continued developing the pcb board
Parts:
- C21, C22, C23: value 47uF 35V X7R MLCC -> 22uF 25V X5R MLCC; footprint Capacitor_SMD:C_2220_5750Metric -> Capacitor_SMD:C_1210_3225Metric; JLCPCB part C3873016 -> C12891

Commit message: finnished component placement
Parts:
- removed D4, D5, D6: BAT165, Drone_components:BAT165, symbol Drone_components:BAT165
- added D4, D5, D6: RB520S30, Drone_components:RB520S30, symbol Drone_components:RB520S30
- C27, C29, C30: value 0.47uF 25V X7R MLCC -> 1uF 25V X5R MLCC; footprint Capacitor_SMD:C_0603_1608Metric -> Capacitor_SMD:C_0402_1005Metric; JLCPCB part C1623 -> C52923
- C28: value 4.7uF 25V X7R MLCC -> 10uF 25V X5R MLCC; footprint Capacitor_SMD:C_1206_3216Metric -> Capacitor_SMD:C_0603_1608Metric; JLCPCB part C29823 -> C96446
Connections:
- net VCC: now also D4.2, D5.2, D6.2
- net at C27.1, U6.20 (VB1): now also D4.1
- net at C30.1, U6.14 (VB3): now also D6.1
- net at C29.1, U6.17 (VB2): now also D5.1

Commit message: replaced some of the schematics
Parts:
- removed Q10, Q11, Q12, Q7, Q8, Q9: BSC016N04LS, Drone_components:BSC016N04LS, symbol Drone_components:BSC016N04LS
- added Q10, Q11, Q12, Q7, Q8, Q9: BSC009NE2LS5IATMA1, Drone_components:BSC093N04LSGATMA1, symbol Drone_components:BSC009NE2LS5IATMA1
- C21, C22, C23: footprint Capacitor_SMD:C_1210_3225Metric -> Capacitor_SMD:C_0805_2012Metric; JLCPCB part C12891 -> C45783
- R14, R16, R17, R18, R19, R20: value 33 -> 47
Connections:
- net GND: now also Q10.1, Q10.2, Q10.3, Q12.1, Q12.2, Q12.3, Q8.1, Q8.2, Q8.3
- net VCC: now also Q11.5, Q7.5, Q9.5
- net VS1: now also Q7.1, Q7.2, Q7.3, Q8.5
- net VS2: now also Q10.5, Q9.1, Q9.2, Q9.3
- net VS3: now also Q11.1, Q11.2, Q11.3, Q12.5
- net at R19.2: now also Q11.4
- net at R17.2: now also Q9.4
- net at R18.2: now also Q10.4
- net at R14.2: now also Q7.4
- net at R16.2: now also Q8.4
- net at R20.2: now also Q12.4
Other:
- moved on the sheet: R14, R16, R17, R18, R19, R20

Commit message: changed some footprints and reconstracted the latout with better gate resistors clearence
Parts:
- R14, R16, R17, R18, R19, R20: value 47 -> 10; footprint Resistor_SMD:R_0402_1005Metric -> Resistor_SMD:R_0201_0603Metric; JLCPCB part C25105 -> C105889
