File: hardware/drone_esc/schematics/esc_4.kicad_sch (KiCad schematic)
At the start: 0 parts

Commit message: finished 4 esc schematics need further refinment of the sheets
Parts:
- added C47, C48, C49: 47uF 35V X7R MLCC, Capacitor_SMD:C_2220_5750Metric, symbol Device:C
- added C50, C51, C52: 10nF 10V X7R MLCC, Capacitor_SMD:C_0402_1005Metric, symbol Device:C
- added C53, C55, C56: 0.47uF 25V X7R MLCC, Capacitor_SMD:C_0603_1608Metric, symbol Device:C
- added C54: 4.7uF 25V X7R MLCC, Capacitor_SMD:C_1206_3216Metric, symbol Device:C
- added D10, D11, D12: BAT165, Drone_components:BAT165, symbol Drone_components:BAT165
- added Q19, Q20, Q21, Q22, Q23, Q24: BSC016N04LS, Drone_components:BSC016N04LS, symbol Drone_components:BSC016N04LS
- added R39, R40, R41, R42, R43, R44: 33, Resistor_SMD:R_0402_1005Metric, symbol Device:R
- added R45, R47, R49: 4.7k, Resistor_SMD:R_0402_1005Metric, symbol Device:R
- added R46, R48, R50: 1k, Resistor_SMD:R_0402_1005Metric, symbol Device:R
- added U10: FD6288Q, Drone_components:FD6288Q, symbol Drone_components:FD6288Q
Connections:
- new net: C55.1, D11.1, U10.17 (VB2)
- new net: C53.1, D10.1, U10.20 (VB1)
- new net: Q23.4, R43.2
- new net: Q20.4, R40.2
- new net: Q19.4, R39.2
- new net: C56.1, D12.1, U10.14 (VB3)
- new net: Q21.4, R41.2
- new net: Q24.4, R44.2
- new net: Q22.4, R42.2
- new net GND: C47.2, C48.2, C49.2, C50.2, C51.2, C52.2, C54.1, Q20.1-3, Q22.1-3, Q24.1-3, R46.1, R48.1, R50.1, U10.25 (EXP), U10.6 (COM)
- new net HIN4A: U10.22 (HIN1)
- new net HIN4B: U10.23 (HIN2)
- new net HIN4C: U10.24 (HIN3)
- new net HO1: R39.1, U10.19 (HO1)
- new net HO2: R41.1, U10.16 (HO2)
- new net HO3: R43.1, U10.13 (HO3)
- new net LIN4A: U10.1 (LIN1)
- new net LIN4B: U10.2 (LIN2)
- new net LIN4C: U10.3 (LIN3)
- new net LO1: R40.1, U10.11 (LO1)
- new net LO2: R42.1, U10.10 (LO2)
- new net LO3: R44.1, U10.9 (LO3)
- new net VCC: C47.1, C48.1, C49.1, C54.2, D10.2, D11.2, D12.2, Q19.5-8, Q21.5-8, Q23.5-8, U10.4 (VCC)
- new net VS1: C53.2, Q19.1-3, Q20.5-8, R45.2, U10.18 (VS1)
- new net VS2: C55.2, Q21.1-3, Q22.5-8, R47.2, U10.15 (VS2)
- new net VS3: C56.2, Q23.1-3, Q24.5-8, R49.2, U10.12 (VS3)
- new net VSense4A: C50.1, R45.1, R46.2
- new net VSense4B: C51.1, R47.1, R48.2
- new net VSense4C: C52.1, R49.1, R50.2

Commit message: continued developing the pcb board
Parts:
- C47, C48, C49: value 47uF 35V X7R MLCC -> 22uF 25V X5R MLCC; footprint Capacitor_SMD:C_2220_5750Metric -> Capacitor_SMD:C_1210_3225Metric; JLCPCB part C3873016 -> C12891
Changed lines of the file:
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@@
 			)
 		)
-		(property "Value" "47uF 35V X7R MLCC"
+		(property "Value" "22uF 25V X5R MLCC"
 			(at 107.95 90.1699 0)
 			(effects
@@
 			)
 		)
-		(property "Footprint" "Capacitor_SMD:C_2220_5750Metric"
+		(property "Footprint" "Capacitor_SMD:C_1210_3225Metric"
 			(at 105.1052 92.71 0)
 			(effects
@@
 			)
 		)
-		(property "JLCPCB part" "C3873016"
+		(property "JLCPCB part" "C12891"
 			(at 104.14 88.9 0)
 			(effects
@@
 	)
 	(symbol
+		(lib_id "Device:C")
+		(at 104.14 35.56 0)
+		(unit 1)
+		(exclude_from_sim no)
+		(in_bom yes)
+		(on_board yes)
+		(dnp no)
+		(fields_autoplaced yes)
+		(property "Reference" "C47"
+			(at 107.95 34.2899 0)
+			(effects
+				(font
+					(size 1.27 1.27)
+				)
+				(justify left)
+			)
+		)
+		(property "Value" "22uF 25V X5R MLCC"
+			(at 107.95 36.8299 0)
+			(effects
+				(font
+					(size 1.27 1.27)
+				)
+				(justify left)
+			)
+		)
+		(property "Footprint" "Capacitor_SMD:C_1210_3225Metric"
+			(at 105.1052 39.37 0)
+			(effects
+				(font
+					(size 1.27 1.27)
+				)
+				(hide yes)
+			)
+		)
+		(property "Datasheet" "~"
+			(at 104.14 35.56 0)
+			(effects
+				(font
+					(size 1.27 1.27)
+				)
+				(hide yes)
+			)
+		)
+		(property "Description" "Unpolarized capacitor"
+			(at 104.14 35.56 0)
+			(effects
+				(font
+					(size 1.27 1.27)
+				)
+				(hide yes)
+			)
+		)
+		(property "JLCPCB part" "C12891"
+			(at 104.14 35.56 0)
+			(effects
+				(font
+					(size 1.27 1.27)
+				)
+				(hide yes)
+			)
+		)
+		(pin "2"
+		)
+		(pin "1"
+		)
+		(instances
+			(project "drone_esc"
+				(path "/b5a13fd4-6868-4fff-a56c-eae40f1d53c7/8c7f729c-8a7e-42fc-ba88-d14a0a817b1c"
+					(reference "C47")
+					(unit 1)
+				)
+			)
+		)
+	)
+	(symbol
 		(lib_id "Device:R")
 		(at 105.41 110.49 180)
@@
 	)
 	(symbol
-		(lib_id "Device:C")
-		(at 104.14 35.56 0)
-		(unit 1)
-		(exclude_from_sim no)
-		(in_bom yes)
-		(on_board yes)
-		(dnp no)
-		(fields_autoplaced yes)
-		(property "Reference" "C47"
-			(at 107.95 34.2899 0)
-			(effects
-				(font
-					(size 1.27 1.27)
-				)
-				(justify left)
-			)
-		)
-		(property "Value" "47uF 35V X7R MLCC"
-			(at 107.95 36.8299 0)
-			(effects
-				(font
-					(size 1.27 1.27)
-				)
-				(justify left)
-			)
-		)
-		(property "Footprint" "Capacitor_SMD:C_2220_5750Metric"
-			(at 105.1052 39.37 0)
-			(effects
-				(font
-					(size 1.27 1.27)
-				)
-				(hide yes)
-			)
-		)
-		(property "Datasheet" "~"
-			(at 104.14 35.56 0)
-			(effects
-				(font
-					(size 1.27 1.27)
-				)
-				(hide yes)
-			)
-		)
-		(property "Description" "Unpolarized capacitor"
-			(at 104.14 35.56 0)
-			(effects
-				(font
-					(size 1.27 1.27)
-				)
-				(hide yes)
-			)
-		)
-		(property "JLCPCB part" "C3873016"
-			(at 104.14 35.56 0)
-			(effects
-				(font
-					(size 1.27 1.27)
-				)
-				(hide yes)
-			)
-		)
-		(pin "2"
-		)
-		(pin "1"
-		)
-		(instances
-			(project "drone_esc"
-				(path "/b5a13fd4-6868-4fff-a56c-eae40f1d53c7/8c7f729c-8a7e-42fc-ba88-d14a0a817b1c"
-					(reference "C47")
-					(unit 1)
-				)
-			)
-		)
-	)
-	(symbol
 		(lib_id "Drone_components:BSC016N04LS")
 		(at 78.74 148.59 0)
@@
 	)
 	(symbol
-		(lib_id "Device:C")
-		(at 104.14 143.51 0)
-		(unit 1)
-		(exclude_from_sim no)
-		(in_bom yes)
-		(on_board yes)
-		(dnp no)
-		(fields_autoplaced yes)
-		(property "Reference" "C49"
-			(at 107.95 142.2399 0)
-			(effects
-				(font
-					(size 1.27 1.27)
-				)
-				(justify left)
-			)
-		)
-		(property "Value" "47uF 35V X7R MLCC"
-			(at 107.95 144.7799 0)
-			(effects
-				(font
-					(size 1.27 1.27)
-				)
-				(justify left)
-			)
-		)
-		(property "Footprint" "Capacitor_SMD:C_2220_5750Metric"
-			(at 105.1052 147.32 0)
-			(effects
-				(font
-					(size 1.27 1.27)
-				)
-				(hide yes)
-			)
-		)
-		(property "Datasheet" "~"
-			(at 104.14 143.51 0)
-			(effects
-				(font
-					(size 1.27 1.27)
-				)
-				(hide yes)
-			)
-		)
-		(property "Description" "Unpolarized capacitor"
-			(at 104.14 143.51 0)
-			(effects
-				(font
-					(size 1.27 1.27)
-				)
-				(hide yes)
-			)
-		)
-		(property "JLCPCB part" "C3873016"
-			(at 104.14 143.51 0)
-			(effects
-				(font
-					(size 1.27 1.27)
-				)
-				(hide yes)
-			)
-		)
-		(pin "2"
-		)
-		(pin "1"
-		)
-		(instances
-			(project "drone_esc"
-				(path "/b5a13fd4-6868-4fff-a56c-eae40f1d53c7/8c7f729c-8a7e-42fc-ba88-d14a0a817b1c"
-					(reference "C49")
-					(unit 1)
-				)
-			)
-		)
-	)
-	(symbol
 		(lib_id "Device:R")
 		(at 64.77 171.45 90)
@@
 					(unit 1)
 				)
+			)
+		)
+	)
+	(symbol
+		(lib_id "Device:C")
+		(at 104.14 143.51 0)
+		(unit 1)
+		(exclude_from_sim no)
+		(in_bom yes)
+		(on_board yes)
+		(dnp no)
+		(fields_autoplaced yes)
+		(property "Reference" "C49"
+			(at 107.95 142.2399 0)
+			(effects
+				(font
+					(size 1.27 1.27)
+				)
+				(justify left)
+			)
+		)
+		(property "Value" "22uF 25V X5R MLCC"
+			(at 107.95 144.7799 0)
+			(effects
+				(font
+					(size 1.27 1.27)
+				)
+				(justify left)
+			)
+		)
+		(property "Footprint" "Capacitor_SMD:C_1210_3225Metric"
+			(at 105.1052 147.32 0)
+			(effects
+				(font
+					(size 1.27 1.27)
+				)
+				(hide yes)
+			)
+		)
+		(property "Datasheet" "~"
+			(at 104.14 143.51 0)
+			(effects
+				(font
+					(size 1.27 1.27)
+				)
+				(hide yes)
+			)
+		)
+		(property "Description" "Unpolarized capacitor"
+			(at 104.14 143.51 0)
+			(effects
+				(font
+					(size 1.27 1.27)
+				)
+				(hide yes)
+			)
+		)
+		(property "JLCPCB part" "C12891"
+			(at 104.14 143.51 0)
+			(effects
+				(font
+					(size 1.27 1.27)
+				)
+				(hide yes)
+			)
+		)
+		(pin "2"
+		)
+		(pin "1"
+		)
+		(instances
+			(project "drone_esc"
+				(path "/b5a13fd4-6868-4fff-a56c-eae40f1d53c7/8c7f729c-8a7e-42fc-ba88-d14a0a817b1c"
+					(reference "C49")
+					(unit 1)
+				)

Commit message: finnished component placement
Parts:
- removed D10, D11, D12: BAT165, Drone_components:BAT165, symbol Drone_components:BAT165
- added D10, D11, D12: RB520S30, Drone_components:RB520S30, symbol Drone_components:RB520S30
- C53, C55, C56: value 0.47uF 25V X7R MLCC -> 1uF 25V X5R MLCC; footprint Capacitor_SMD:C_0603_1608Metric -> Capacitor_SMD:C_0402_1005Metric; JLCPCB part C1623 -> C52923
- C54: value 4.7uF 25V X7R MLCC -> 10uF 25V X5R MLCC; footprint Capacitor_SMD:C_1206_3216Metric -> Capacitor_SMD:C_0603_1608Metric; JLCPCB part C29823 -> C96446
Connections:
- net VCC: now also D10.2, D11.2, D12.2
- net at C55.1, U10.17 (VB2): now also D11.1
- net at C53.1, U10.20 (VB1): now also D10.1
- net at C56.1, U10.14 (VB3): now also D12.1

Commit message: replaced some of the schematics
Parts:
- removed Q19, Q20, Q21, Q22, Q23, Q24: BSC016N04LS, Drone_components:BSC016N04LS, symbol Drone_components:BSC016N04LS
- added Q19, Q20, Q21, Q22, Q23, Q24: BSC009NE2LS5IATMA1, Drone_components:BSC093N04LSGATMA1, symbol Drone_components:BSC009NE2LS5IATMA1
- C47, C48, C49: footprint Capacitor_SMD:C_1210_3225Metric -> Capacitor_SMD:C_0805_2012Metric; JLCPCB part C12891 -> C45783
- R39, R40, R41, R42, R43, R44: value 33 -> 47
Connections:
- net GND: now also Q20.1, Q20.2, Q20.3, Q22.1, Q22.2, Q22.3, Q24.1, Q24.2, Q24.3
- net VCC: now also Q19.5, Q21.5, Q23.5
- net VS1: now also Q19.1, Q19.2, Q19.3, Q20.5
- net VS2: now also Q21.1, Q21.2, Q21.3, Q22.5
- net VS3: now also Q23.1, Q23.2, Q23.3, Q24.5
- net at R43.2: now also Q23.4
- net at R40.2: now also Q20.4
- net at R39.2: now also Q19.4
- net at R41.2: now also Q21.4
- net at R44.2: now also Q24.4
- net at R42.2: now also Q22.4
Other:
- moved on the sheet: R39, R40, R41, R42, R43, R44

Commit message: changed some footprints and reconstracted the latout with better gate resistors clearence
Parts:
- R39, R40, R41, R42, R43, R44: value 47 -> 10; footprint Resistor_SMD:R_0402_1005Metric -> Resistor_SMD:R_0201_0603Metric; JLCPCB part C25105 -> C105889
